File: hardware/pmod-apa102/pmod-apa102.sch (EAGLE design)
At the start: 9 parts, among them J4 RA 6Pin SMD

Commit message: APA102 PMD as submitted to Oshpark (minor silk fixups)
Parts:
- J4: device SparkFun-Connectors:CONN_06SMD -> mechanical:CONN_06SMD
Changed lines of the file:
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@@
 <part name="GND4" library="supply1" deviceset="GND" device=""/>
 <part name="GND5" library="supply1" deviceset="GND" device=""/>
-<part name="J4" library="SparkFun-Connectors" deviceset="CONN_06" device="SMD" value="RA 6Pin SMD"/>
+<part name="J4" library="mechanical" deviceset="CONN_06" device="SMD" value="RA 6Pin SMD"/>
 <part name="P+6" library="supply1" deviceset="+5V" device=""/>
 <part name="GND6" library="supply1" deviceset="GND" device=""/>
