File: hardware/pmod-level-conv/pmod-level-conv.sch (EAGLE design)
At the start: 6 parts, among them J1 PMOD_PLUG1, J2 PMOD_SOCKET1, J3 VCC, U1 TXB0108PWR

Commit message: pmod-level-conv : fixed NC OE
Connections:
- net VCCIO: now also U1.OE
Changed lines of the file:
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@@
 <pinref part="U1" gate="G$1" pin="VCCA"/>
 <pinref part="VCC2" gate="G$1" pin="VCCIO"/>
-<wire x1="33.02" y1="22.86" x2="33.02" y2="27.94" width="0.1524" layer="91"/>
+<wire x1="33.02" y1="22.86" x2="33.02" y2="25.4" width="0.1524" layer="91"/>
+<pinref part="U1" gate="G$1" pin="OE"/>
+<wire x1="33.02" y1="25.4" x2="33.02" y2="27.94" width="0.1524" layer="91"/>
+<wire x1="20.32" y1="15.24" x2="17.78" y2="15.24" width="0.1524" layer="91"/>
+<wire x1="17.78" y1="15.24" x2="17.78" y2="25.4" width="0.1524" layer="91"/>
+<wire x1="17.78" y1="25.4" x2="33.02" y2="25.4" width="0.1524" layer="91"/>
+<junction x="33.02" y="25.4"/>
 </segment>
 </net>
