File: hardware/pmod-16x16led/pmod-16x16led.kicad_pcb (KiCad board)
At the start: 2 copper layers, 31 x 40 mm, 13 parts, among them J1 Conn_01x06, U1 74HC595, U2 74HC595, U3 74HC595, U4 74HC595

Commit message: pmod-16x16led: Apr2020 version as submitted to oshpark
Parts:
- added G***: LOGO, pmod-16x16led:mask_600, F.Cu at (157.8, 85.8)
Routing:
- net /DATA: track 61.4 -> 68.7 mm
- net GND: track 17.8 -> 11.5 mm, vias 13 -> 9
- net /DATA-A16: track 66.5 -> 61.1 mm
- net /A4: track 18.6 -> 23.8 mm
- net /C16: track 12.7 -> 16.2 mm
- net /A7: track 14.8 -> 11.7 mm
- net /C15: track 11.5 -> 14.5 mm
- net /A15: track 11.2 -> 14.2 mm
- net /A5: track 8.85 -> 11.6 mm
- net /C14: track 9.99 -> 12.5 mm
- net /C13: track 8.49 -> 10.8 mm
- net /C12: track 6.30 -> 8.49 mm
- net /C4: track 9.73 -> 11.7 mm
- net /A14: track 6.20 -> 8.02 mm
- net +3V3: track 127.4 -> 129.2 mm, vias 7 -> 8
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Other:
- board size 31 x 40 mm -> 37.5 x 43.2 mm
